Commit message: Add ROS 2 Gazebo validation workflow

File: robots/my_robot_2kg_payload.urdf (robot description, URDF)
Before this commit: robot envelope_test_robot, 5 links, 4 joints
Links:
- added link payload_2kg, mass 2.0; collision box size=0.20 0.20 0.10; visual box size=0.20 0.20 0.10
Joints:
- added joint payload_fixed_joint: type fixed, parent base_link, child payload_2kg, origin xyz=0 0 0.15 rpy=0 0 0

File: robots/my_robot_5_44kg_payload.urdf (robot description, URDF)
Before this commit: robot envelope_test_robot, 5 links, 4 joints
Links:
- added link payload_5_44kg, mass 5.44; collision box size=0.30 0.30 0.22; visual box size=0.30 0.30 0.22
Joints:
- added joint payload_5_44kg_fixed_joint: type fixed, parent base_link, child payload_5_44kg, origin xyz=0 0 0.21 rpy=0 0 0

File: robots/my_robot_5kg_payload.urdf (robot description, URDF)
Before this commit: robot envelope_test_robot, 5 links, 4 joints
Links:
- added link payload_5kg, mass 5.0; collision box size=0.30 0.30 0.20; visual box size=0.30 0.30 0.20
Joints:
- added joint payload_5kg_fixed_joint: type fixed, parent base_link, child payload_5kg, origin xyz=0 0 0.20 rpy=0 0 0

File: robots/my_robot_6kg_payload.urdf (robot description, URDF)
Before this commit: robot envelope_test_robot, 5 links, 4 joints
Links:
- added link payload_6kg, mass 6.0; collision box size=0.30 0.30 0.24; visual box size=0.30 0.30 0.24
Joints:
- added joint payload_6kg_fixed_joint: type fixed, parent base_link, child payload_6kg, origin xyz=0 0 0.22 rpy=0 0 0
